File: hardware/mainboard-atlas/Mainboard-ATLAS.kicad_pcb (KiCad board)
At the start: 2 copper layers, 100 x 80 mm, 25 parts, among them J1 J1 // 24V IN, J2 Conn_01x04, J3 Conn_01x04, J7 Conn_01x02, J9 3.3V OUT, U1 // TSR_1-2450 TSR_1-2450

Commit message: fix(hardware): H1 annotation-debt fix on Mainboard-ATLAS board
Board adopts schematic references (designer ruling: schematic owns refs):
LOADCELL->J4 (net proof: J4.1 on Net-(HX1-A+)), HX711->HX1,
ENDSTOP1->J5 / ENDSTOP2->J6 and TMC2209x2->TMC1/TMC2 (pairings proven by
pin-net set equality vs sch export netlist, never by position), 10 refs
stripped of ' // <value>' corruption (C1-C6, D1, F1, U1), REF** x4 named
H1..H4 (exclude_from_bom/pos already present).

Also fixes debt exposed once refs matched:
- 16x board Datasheet field '~' aligned to schematic empty (FR-007)
- J1 board Value 'J1 // 24V IN' -> schematic value Screw_Terminal_01x02
  (FR-008); the clean long value clipped the board edge on silk
  (silk_edge_clearance warning), so the J1 Value field layer moves
  F.SilkS->F.Fab (display metadata, no geometry).

Invariant: pad-uuid->net map byte-identical pre/post (script-asserted);
schematic and .kicad_pro untouched (diff-verified). Fingerprint ledger
drifts exactly parity 44->4 (4 board-only mounting holes, no KiCad 10
suppression exists) and gerber_sha (intended silk change); DRC/ERC/counts
unchanged. Spec: specs/H1-atlas-annotation-debt/
Parts:
- C1: renamed from C1 // 100µF
- C2: renamed from C2 // 100nF
- C3: renamed from C3 // 100µF
- C4: renamed from C4 // 100nF
- C5: renamed from C5 // 100µF
- C6: renamed from C6 // 100nF
- D1: renamed from D1 // 1N5819
- F1: renamed from F1 // Fuse 2A T
- J1: value J1 // 24V IN -> Screw_Terminal_01x02
- U1: renamed from U1 // TSR_1-2450
- renumbered REF** to H1, REF** to H2, REF** to H3, REF** to H4, HX711 to HX1, LOADCELL to J4, ENDSTOP1 to J5, ENDSTOP2 to J6, TMC2209 to TMC1, TMC2209 to TMC2
Changed lines of the file:
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@@
 		(descr "Pololu Breakout 16-pin 15.2x20.3mm 0.6x0.8")
 		(tags "Pololu Breakout")
-		(property "Reference" "TMC2209"
+		(property "Reference" "TMC1"
 			(at 6.35 17.41 90)
 			(layer "F.SilkS")
@@
 			)
 		)
-		(property "Datasheet" "~"
+		(property "Datasheet" ""
 			(at 0 0 0)
 			(layer "F.Fab")
@@
 		(descr "C, Disc series, Radial, pin pitch=5.00mm, diameter*width=5*2.5mm^2, Capacitor, http://cdn-reichelt.de/documents/datenblatt/B300/DS_KERKO_TC.pdf")
 		(tags "C Disc series Radial pin pitch 5.00mm diameter 5mm width 2.5mm Capacitor")
-		(property "Reference" "C6 // 100nF"
+		(property "Reference" "C6"
 			(at 2.5 -2.5 90)
 			(layer "F.SilkS")
@@
 			)
 		)
-		(property "Datasheet" "~"
+		(property "Datasheet" ""
 			(at 0 0 90)
 			(layer "F.Fab")
@@
 		(layer "F.Cu")
 		(at 125.65 73 90)
-		(property "Reference" "HX711"
+		(property "Reference" "HX1"
 			(at 10 6.35 0)
 			(unlocked yes)
@@
 		(descr "C, Disc series, Radial, pin pitch=5.00mm, diameter*width=5*2.5mm^2, Capacitor, http://cdn-reichelt.de/documents/datenblatt/B300/DS_KERKO_TC.pdf")
 		(tags "C Disc series Radial pin pitch 5.00mm diameter 5mm width 2.5mm Capacitor")
-		(property "Reference" "C4 // 100nF"
+		(property "Reference" "C4"
 			(at 2 -2.5 90)
 			(layer "F.SilkS")
@@
 			)
 		)
-		(property "Datasheet" "~"
+		(property "Datasheet" ""
 			(at 0 0 90)
 			(layer "F.Fab")
@@
 		(descr "DCDC-Converter, TRACO, TSR 1-xxxx")
 		(tags "DCDC-Converter TRACO TSR-1")
-		(property "Reference" "U1 // TSR_1-2450"
+		(property "Reference" "U1"
 			(at 2.5425 3.6275 0)
 			(layer "F.SilkS")
@@
 		(descr "CP, Radial series, Radial, pin pitch=3.50mm, diameter=8mm, height=12mm, Electrolytic Capacitor")
 		(tags "CP Radial series Radial pin pitch 3.50mm diameter 8mm height 12mm Electrolytic Capacitor")
-		(property "Reference" "C3 // 100µF"
+		(property "Reference" "C3"
 			(at 7.49 0.2 90)
 			(layer "F.SilkS")
@@
 			)
 		)
-		(property "Datasheet" "~"
+		(property "Datasheet" ""
 			(at 0 0 0)
 			(layer "F.Fab")
@@
 		(descr "Diode, DO-41_SOD81 series, Axial, Horizontal, pin pitch=10.16mm, length*diameter=5.2*2.7mm^2, https://www.diodes.com/assets/Package-Files/DO-41-Plastic.pdf")
 		(tags "Diode DO-41_SOD81 series Axial Horizontal pin pitch 10.16mm  length 5.2mm diameter 2.7mm")
-		(property "Reference" "D1 // 1N5819"
+		(property "Reference" "D1"
 			(at 5.08 -2.47 90)
 			(layer "F.SilkS")
@@
 			)
 		)
-		(property "Datasheet" "~"
+		(property "Datasheet" ""
 			(at 0 0 90)
 			(layer "F.Fab")
@@
 		(descr "Fuseholder horizontal open, 5x20mm, 500V, 16A, Schurter 0031.8201, https://us.schurter.com/bundles/snceschurter/epim/_ProdPool_/newDS/en/typ_OGN.pdf")
 		(tags "Fuseholder horizontal open 5x20 Schurter 0031.8201")
-		(property "Reference" "F1 // Fuse 2A T"
+		(property "Reference" "F1"
 			(at 11.25 -6 0)
 			(layer "F.SilkS")
@@
 			)
 		)
-		(property "Datasheet" "~"
+		(property "Datasheet" ""
 			(at 0 0 0)
 			(unlocked yes)
@@
 		(descr "JST XH series connector, B3B-XH-A (http://www.jst-mfg.com/product/pdf/eng/eXH.pdf), generated with kicad-footprint-generator")
 		(tags "connector JST XH vertical")
-		(property "Reference" "ENDSTOP1"
+		(property "Reference" "J5"
 			(at 2.774 6.898 0)
 			(layer "F.SilkS")
@@
 			)
 		)
-		(property "Datasheet" "~"
+		(property "Datasheet" ""
 			(at 0 0 0)
 			(layer "F.Fab")
@@
 		(descr "JST XH series connector, B3B-XH-A (http://www.jst-mfg.com/product/pdf/eng/eXH.pdf), generated with kicad-footprint-generator")
 		(tags "connector JST XH vertical")
-		(property "Reference" "ENDSTOP2"
+		(property "Reference" "J6"
 			(at 2.53 6.915 0)
 			(layer "F.SilkS")
@@
 			)
 		)
-		(property "Datasheet" "~"
+		(property "Datasheet" ""
 			(at 0 0 0)
 			(layer "F.Fab")
@@
 		(descr "JST XH series connector, B4B-XH-A (http://www.jst-mfg.com/product/pdf/eng/eXH.pdf), generated with kicad-footprint-generator")
 		(tags "connector JST XH vertical")
-		(property "Reference" "LOADCELL"
+		(property "Reference" "J4"
 			(at -7.25 -0.95 90)
 			(layer "F.SilkS")
@@
 			)
 		)
-		(property "Datasheet" "~"
+		(property "Datasheet" ""
 			(at 0 0 90)
 			(layer "F.Fab")
@@
 		(descr "Mounting Hole 3.2mm, M3, no annular, generated by kicad-footprint-generator mountinghole.py")
 		(tags "mountinghole M3")
-		(property "Reference" "REF**"
+		(property "Reference" "H3"
 			(at 0 -4.15 0)
 			(layer "F.SilkS")
@@
 		(descr "Mounting Hole 3.2mm, M3, no annular, generated by kicad-footprint-generator mountinghole.py")
 		(tags "mountinghole M3")
-		(property "Reference" "REF**"
+		(property "Reference" "H4"
 			(at 0 -4.15 0)
 			(layer "F.SilkS")
@@
 		(descr "CP, Radial series, Radial, pin pitch=3.50mm, diameter=8mm, height=12mm, Electrolytic Capacitor")
 		(tags "CP Radial series Radial pin pitch 3.50mm diameter 8mm height 12mm Electrolytic Capacitor")
-		(property "Reference" "C5 // 100µF"
+		(property "Reference" "C5"
 			(at 0.99 -5.35 90)
 			(layer "F.SilkS")
@@
 			)
 		)
-		(property "Datasheet" "~"
+		(property "Datasheet" ""
 			(at 0 0 90)
 			(layer "F.Fab")
@@
 			)
 		)
-		(property "Datasheet" "~"
+		(property "Datasheet" ""
 			(at 0 0 90)
 			(layer "F.Fab")
@@
 		(descr "Mounting Hole 3.2mm, M3, no annular, generated by kicad-footprint-generator mountinghole.py")
 		(tags "mountinghole M3")
-		(property "Reference" "REF**"
+		(property "Reference" "H1"
 			(at 0 -4.15 0)
 			(layer "F.SilkS")
@@
 		(descr "Mounting Hole 3.2mm, M3, no annular, generated by kicad-footprint-generator mountinghole.py")
 		(tags "mountinghole M3")
-		(property "Reference" "REF**"
+		(property "Reference" "H2"
 			(at 0 -4.15 0)
 			(layer "F.SilkS")
@@
 			)
 		)
-		(property "Datasheet" "~"
+		(property "Datasheet" ""
 			(at 0 0 0)
 			(layer "F.Fab")
@@
 		(descr "CP, Radial series, Radial, pin pitch=3.50mm, diameter=8mm, height=12mm, Electrolytic Capacitor")
 		(tags "CP Radial series Radial pin pitch 3.50mm diameter 8mm height 12mm Electrolytic Capacitor")
-		(property "Reference" "C1 // 100µF"
+		(property "Reference" "C1"
 			(at 1.75 -5.25 90)
 			(layer "F.SilkS")
@@
 			)
 		)
-		(property "Datasheet" "~"
+		(property "Datasheet" ""
 			(at 0 0 90)
 			(layer "F.Fab")
@@
 			)
 		)
-		(property "Datasheet" "~"
+		(property "Datasheet" ""
 			(at 0 0 0)
 			(layer "F.Fab")
@@
 			)
 		)
-		(property "Value" "J1 // 24V IN"
+		(property "Value" "Screw_Terminal_01x02"
 			(at 10.47 0.4775 180)
-			(layer "F.SilkS")
+			(layer "F.Fab")
 			(effects
 				(font
@@
 			)
 		)
-		(property "Datasheet" "~"
+		(property "Datasheet" ""
 			(at 0 0 90)
 			(layer "F.Fab")
@@
 		(descr "Pololu Breakout 16-pin 15.2x20.3mm 0.6x0.8")
 		(tags "Pololu Breakout")
-		(property "Reference" "TMC2209"
+		(property "Reference" "TMC2"
 			(at 6.35 17.62 90)
 			(layer "F.SilkS")
@@
 		(descr "C, Disc series, Radial, pin pitch=5.00mm, diameter*width=5*2.5mm^2, Capacitor, http://cdn-reichelt.de/documents/datenblatt/B300/DS_KERKO_TC.pdf")
 		(tags "C Disc series Radial pin pitch 5.00mm diameter 5mm width 2.5mm Capacitor")
-		(property "Reference" "C2 // 100nF"
+		(property "Reference" "C2"
 			(at 0.5 2.63 90)
 			(layer "F.SilkS")
@@
 			)
 		)
-		(property "Datasheet" "~"
+		(property "Datasheet" ""
 			(at 0 0 90)
 			(layer "F.Fab")
